File: eagle/disturber85.brd (EAGLE design)
At the start: 50 x 50 mm, 14 parts, among them J6 455-1750-1-ND, J7 455-1750-1-ND, J8 455-1750-1-ND, U1 ATTINY85, U2 ATTINY85-20P, U3 ATTINY85, U4 ATTINY85-20P

Commit message: Panelized
Parts:
- added SV3, SV4: (no value), con-lstb:MA04-1
Connections:
- net N$1: now also SV3.1, SV3.2
- net N$15: now also SV4.3, SV4.4
- net N$7: now also SV3.3, SV3.4
- net N$9: now also SV4.1, SV4.2
Routing:
- net N$9: track 69.0 -> 75.8 mm
- net N$7: track 37.3 -> 43.7 mm
- net N$1: track 64.1 -> 70.5 mm
- net N$15: track 39.7 -> 45.6 mm
Changed lines of the file:
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@@
 <attribute name="PROD_ID" value="XXX-00000" x="43.18" y="74.93" size="1.778" layer="27" display="off"/>
+</element>
+<element name="SV3" library="con-lstb" library_urn="urn:adsk.eagle:library:162" package="MA04-1" package3d_urn="urn:adsk.eagle:package:8337/1" value="" x="2.54" y="90.17" smashed="yes" rot="R90">
+<attribute name="MF" value="" x="2.54" y="90.17" size="1.778" layer="27" rot="R90" display="off"/>
+<attribute name="MPN" value="" x="2.54" y="90.17" size="1.778" layer="27" rot="R90" display="off"/>
+<attribute name="OC_FARNELL" value="unknown" x="2.54" y="90.17" size="1.778" layer="27" rot="R90" display="off"/>
+<attribute name="OC_NEWARK" value="unknown" x="2.54" y="90.17" size="1.778" layer="27" rot="R90" display="off"/>
+<attribute name="VALUE" x="0.889" y="90.805" size="1.27" layer="27" ratio="10" rot="R90"/>
+</element>
+<element name="SV4" library="con-lstb" library_urn="urn:adsk.eagle:library:162" package="MA04-1" package3d_urn="urn:adsk.eagle:package:8337/1" value="" x="3.81" y="64.77" smashed="yes" rot="R90">
+<attribute name="MF" value="" x="3.81" y="64.77" size="1.778" layer="27" rot="R90" display="off"/>
+<attribute name="MPN" value="" x="3.81" y="64.77" size="1.778" layer="27" rot="R90" display="off"/>
+<attribute name="OC_FARNELL" value="unknown" x="3.81" y="64.77" size="1.778" layer="27" rot="R90" display="off"/>
+<attribute name="OC_NEWARK" value="unknown" x="3.81" y="64.77" size="1.778" layer="27" rot="R90" display="off"/>
+<attribute name="VALUE" x="2.159" y="65.405" size="1.27" layer="27" ratio="10" rot="R90"/>
 </element>
 </elements>
@@
 <wire x1="6.4008" y1="88.6968" x2="6.35" y2="88.9" width="0.762" layer="16"/>
 <via x="21.9456" y="88.2396" extent="1-16" drill="0.35"/>
+<contactref element="SV3" pad="2"/>
+<contactref element="SV3" pad="1"/>
+<wire x1="2.7432" y1="88.6968" x2="2.7432" y2="86.4108" width="0.762" layer="1"/>
+<wire x1="2.7432" y1="88.6968" x2="2.54" y2="88.9" width="0.762" layer="1"/>
+<wire x1="5.9436" y1="86.4108" x2="2.7432" y2="86.4108" width="0.762" layer="1"/>
+<wire x1="2.7432" y1="86.4108" x2="2.54" y2="86.36" width="0.762" layer="1"/>
+<wire x1="5.9436" y1="86.4108" x2="6.35" y2="86.36" width="0.762" layer="1"/>
 </signal>
 <signal name="N$2">
@@
 <wire x1="20.1168" y1="80.01" x2="20.32" y2="80.01" width="0.762" layer="1"/>
 <wire x1="20.1168" y1="90.5256" x2="20.447" y2="90.805" width="0.762" layer="1"/>
+<contactref element="SV3" pad="4"/>
+<contactref element="SV3" pad="3"/>
+<wire x1="2.7432" y1="93.726" x2="2.7432" y2="91.44" width="0.762" layer="1"/>
+<wire x1="2.7432" y1="93.726" x2="2.54" y2="93.98" width="0.762" layer="1"/>
+<wire x1="6.35" y1="91.44" x2="2.7432" y2="91.44" width="0.762" layer="1"/>
+<wire x1="2.7432" y1="91.44" x2="2.54" y2="91.44" width="0.762" layer="1"/>
 </signal>
 <signal name="N$8">
@@
 <wire x1="43.5" y1="62.5" x2="43.18" y2="62.23" width="0.762" layer="16"/>
 <wire x1="25" y1="53.5" x2="25.4" y2="53.34" width="0.762" layer="16"/>
+<contactref element="SV4" pad="2"/>
+<contactref element="SV4" pad="1"/>
+<wire x1="4.1148" y1="63.0936" x2="4.1148" y2="61.2648" width="0.762" layer="1"/>
+<wire x1="4.1148" y1="61.2648" x2="3.81" y2="60.96" width="0.762" layer="1"/>
+<wire x1="4.1148" y1="63.0936" x2="3.81" y2="63.5" width="0.762" layer="1"/>
+<wire x1="7.3152" y1="61.2648" x2="4.1148" y2="61.2648" width="0.762" layer="16"/>
+<wire x1="4.1148" y1="61.2648" x2="3.81" y2="60.96" width="0.762" layer="16"/>
+<wire x1="7.3152" y1="61.2648" x2="7.62" y2="60.96" width="0.762" layer="16"/>
 </signal>
 <signal name="N$10">
@@
 <wire x1="20" y1="53.5" x2="20.32" y2="53.34" width="0.762" layer="1"/>
 <wire x1="7.5" y1="66" x2="7.62" y2="66.04" width="0.762" layer="1"/>
+<contactref element="SV4" pad="4"/>
+<contactref element="SV4" pad="3"/>
+<wire x1="5.4864" y1="66.294" x2="4.1148" y2="66.294" width="0.762" layer="1"/>
+<wire x1="4.1148" y1="66.294" x2="3.81" y2="66.04" width="0.762" layer="1"/>
+<wire x1="5.4864" y1="66.294" x2="5.5" y2="66" width="0.762" layer="1"/>
+<wire x1="3.81" y1="68.58" x2="7.62" y2="68.58" width="0.762" layer="1"/>
 </signal>
 <signal name="N$16">
